File: kicad/FrontPanelControls/PanelControls.kicad_pcb (KiCad board)
At the start: 2 copper layers, 106 x 37.8 mm, 39 parts, among them J1 Conn_02x04_Odd_Even, SW5 ADJ, U1 PCF8591, U2 PCF8574, U3 WS2812D, U4 WS2812D, U5 WS2812D, U6 WS2812D, U7 WS2812D, U8 WS2812D

Commit message: initial changes FrontPanel
Parts:
- added J2: LED_PIN_SELECT, Connector_PinHeader_2.54mm:PinHeader_2x02_P2.54mm_Vertical, B.Cu at (191.3, 149.9)
Connections:
- net GND renamed @DIN
- J1 pad 1: (no net) -> Net-(J1-Pad1)
- U1 pad 11: (no net) -> Net-(U1-Pad11)
- U1 pad 15: (no net) -> Net-(U1-Pad15)
- U2 pad 4: (no net) -> Net-(U2-Pad4)
- U2 pad 5: (no net) -> Net-(U2-Pad5)
- U2 pad 6: (no net) -> Net-(U2-Pad6)
- U2 pad 7: (no net) -> Net-(U2-Pad7)
- U2 pad 9: (no net) -> Net-(U2-Pad9)
- U3 pad 1: (no net) -> Net-(U3-Pad1)
Routing:
- net +5v: track 109.8 -> 207.0 mm
- net @DIN: track 345.5 -> 364.1 mm, vias 10 -> 11
Other:
- board text added: "ZC95-FrontPanel-Analog(back) bkifft v0.1"
- board text removed: "ZC95-FrontPanel-Analog(back) v0.1"
